File: BFCN-2900+/BFCN-2900+.sch (KiCad schematic (older format))
At the start: 3 parts, among them U1 BFCN-2900+, X1 SMA-BU, X2 SMA-BU

Commit message: BFCN-2900+: Some vias, new footprints
Parts:
- removed X1, X2: SMA-BU, MiniCircuits:SMA-BU-P, symbol SMA-BU
- added X1, X2: SMA-F, JueConnectors:SMA-F-THT, symbol SMA-F
Connections:
- net GNDA: now also X1.GND, X2.GND
- net at U1.1 (IN): now also X1.HF
- net at U1.3 (OUT): now also X2.HF
Changed lines of the file:
@@
 LIBS:mc-attenuators
 LIBS:mc-filters
-LIBS:mc-misc
 LIBS:mc-mixers
+LIBS:JueConnectors
+LIBS:BFCN-2900+-cache
 EELAYER 25 0
 EELAYER END
@@
 Comment4 ""
 $EndDescr
-$Comp
-L SMA-BU X1
-U 1 1 575036BC
-P 4950 3600
-F 0 "X1" H 5200 3650 60  0000 L CNN
-F 1 "SMA-BU" H 5200 3550 60  0000 L CNN
-F 2 "MiniCircuits:SMA-BU-P" H 4950 3600 60  0001 C CNN
-F 3 "" H 4950 3600 60  0000 C CNN
-	1    4950 3600
-	-1   0    0    -1
-$EndComp
-$Comp
-L SMA-BU X2
-U 1 1 5750374B
-P 6950 3600
-F 0 "X2" H 7200 3650 60  0000 L CNN
-F 1 "SMA-BU" H 7200 3550 60  0000 L CNN
-F 2 "MiniCircuits:SMA-BU-P" H 6950 3600 60  0001 C CNN
-F 3 "" H 6950 3600 60  0000 C CNN
-	1    6950 3600
-	1    0    0    -1
-$EndComp
 $Comp
 L BFCN-2900+ U1
@@
 Wire Wire Line
 	6550 3600 6750 3600
+$Comp
+L SMA-F X1
+U 1 1 57518E72
+P 4950 3600
+F 0 "X1" H 5200 3650 60  0000 L CNN
+F 1 "SMA-F" H 5200 3550 60  0000 L CNN
+F 2 "JueConnectors:SMA-F-THT" H 4950 3600 60  0001 C CNN
+F 3 "" H 4950 3600 60  0000 C CNN
+	1    4950 3600
+	-1   0    0    -1
+$EndComp
+$Comp
+L SMA-F X2
+U 1 1 57518F01
+P 6950 3600
+F 0 "X2" H 7200 3650 60  0000 L CNN
+F 1 "SMA-F" H 7200 3550 60  0000 L CNN
+F 2 "JueConnectors:SMA-F-THT" H 6950 3600 60  0001 C CNN
+F 3 "" H 6950 3600 60  0000 C CNN
+	1    6950 3600
+	1    0    0    -1
+$EndComp
 $EndSCHEMATC
