File: PMA2-43LN+/PMA2-43LN+.kicad_pcb (KiCad board)
At the start: 2 copper layers, 60 x 30 mm, 23 parts, among them P1 CONN_01X02, U1 PMA2-43LN+, X1 SMA-F, X2 SMA-F

Commit message: PMA2-43LN+: Finalised
Parts:
- added REF**11: VIA-0.3, JueVias:VIA-0.3, F.Cu at (108.7, 100.2)
- added REF**11: VIA-0.3, JueVias:VIA-0.3, F.Cu at (122.5, 108.9)
- added REF**11: VIA-0.3, JueVias:VIA-0.3, F.Cu at (125.1, 108.9)
- added REF**11: VIA-0.3, JueVias:VIA-0.3, F.Cu at (127.6, 108.8)
- added REF**11: VIA-0.3, JueVias:VIA-0.3, F.Cu at (130.2, 109.1)
- added REF**11: VIA-0.3, JueVias:VIA-0.3, F.Cu at (132.7, 110.7)
- added REF**11: VIA-0.3, JueVias:VIA-0.3, F.Cu at (130.2, 110.8)
- added REF**11: VIA-0.3, JueVias:VIA-0.3, F.Cu at (127.6, 111.1)
- added REF**11: VIA-0.3, JueVias:VIA-0.3, F.Cu at (125.1, 110.8)
- added REF**11: VIA-0.3, JueVias:VIA-0.3, F.Cu at (122.5, 110.8)
- added REF**11: VIA-0.3, JueVias:VIA-0.3, F.Cu at (120.5, 108.8)
- added REF**11: VIA-0.3, JueVias:VIA-0.3, F.Cu at (108.7, 105.5)
- added REF**11: VIA-0.3, JueVias:VIA-0.3, F.Cu at (120.5, 111.6)
- added REF**11: VIA-0.3, JueVias:VIA-0.3, F.Cu at (118.5, 111.0)
- added REF**11: VIA-0.3, JueVias:VIA-0.3, F.Cu at (113.7, 108.8)
- added REF**11: VIA-0.3, JueVias:VIA-0.3, F.Cu at (116.2, 109.1)
- added REF**11: VIA-0.3, JueVias:VIA-0.3, F.Cu at (116.2, 111.0)
- added REF**11: VIA-0.3, JueVias:VIA-0.3, F.Cu at (113.7, 111.1)
- added REF**11: VIA-0.3, JueVias:VIA-0.3, F.Cu at (111.1, 109.1)
- added REF**11: VIA-0.3, JueVias:VIA-0.3, F.Cu at (111.1, 110.8)
- added REF**11: VIA-0.3, JueVias:VIA-0.3, F.Cu at (108.6, 110.8)
- added REF**11: VIA-0.3, JueVias:VIA-0.3, F.Cu at (108.6, 109.1)
- added REF**11: VIA-0.3, JueVias:VIA-0.3, F.Cu at (132.6, 105.5)
- added REF**11: VIA-0.3, JueVias:VIA-0.3, F.Cu at (107.2, 108.0)
- added REF**11: VIA-0.3, JueVias:VIA-0.3, F.Cu at (106.6, 110.0)
- added REF**11: VIA-0.3, JueVias:VIA-0.3, F.Cu at (105.8, 106.0)
- added REF**11: VIA-0.3, JueVias:VIA-0.3, F.Cu at (104.8, 108.2)
- added REF**11: VIA-0.3, JueVias:VIA-0.3, F.Cu at (104.8, 104.0)
- added REF**11: VIA-0.3, JueVias:VIA-0.3, F.Cu at (132.6, 100.2)
- added REF**11: VIA-0.3, JueVias:VIA-0.3, F.Cu at (136.4, 107.8)
- added REF**11: VIA-0.3, JueVias:VIA-0.3, F.Cu at (134.2, 106.0)
- added REF**11: VIA-0.3, JueVias:VIA-0.3, F.Cu at (135.2, 103.9)
- added REF**11: VIA-0.3, JueVias:VIA-0.3, F.Cu at (132.7, 108.2)
- added REF**11: VIA-0.3, JueVias:VIA-0.3, F.Cu at (134.5, 108.9)
- added REF**1101: VIA-0.3, JueVias:VIA-0.3, F.Cu at (140.0, 95.0)
- added REF**1102: VIA-0.3, JueVias:VIA-0.3, F.Cu at (140.0, 100.0)
- added REF**1104: VIA-0.3, JueVias:VIA-0.3, F.Cu at (140.0, 110.0)
- added REF**1105: VIA-0.3, JueVias:VIA-0.3, F.Cu at (140.0, 115.0)
- added REF**1112: VIA-0.3, JueVias:VIA-0.3, F.Cu at (145.0, 100.0)
- added REF**1113: VIA-0.3, JueVias:VIA-0.3, F.Cu at (145.0, 105.0)
- added REF**1114: VIA-0.3, JueVias:VIA-0.3, F.Cu at (145.0, 110.0)
- added REF**112: VIA-0.3, JueVias:VIA-0.3, F.Cu at (95.0, 100.0)
- added REF**113: VIA-0.3, JueVias:VIA-0.3, F.Cu at (95.0, 105.0)
- added REF**114: VIA-0.3, JueVias:VIA-0.3, F.Cu at (95.0, 110.0)
- added REF**121: VIA-0.3, JueVias:VIA-0.3, F.Cu at (100.0, 95.0)
- added REF**122: VIA-0.3, JueVias:VIA-0.3, F.Cu at (100.0, 100.0)
- added REF**124: VIA-0.3, JueVias:VIA-0.3, F.Cu at (100.0, 110.0)
- added REF**125: VIA-0.3, JueVias:VIA-0.3, F.Cu at (100.0, 115.0)
- added REF**131: VIA-0.3, JueVias:VIA-0.3, F.Cu at (105.0, 95.0)
- added REF**132: VIA-0.3, JueVias:VIA-0.3, F.Cu at (105.0, 100.0)
- added REF**134: VIA-0.3, JueVias:VIA-0.3, F.Cu at (105.0, 110.0)
- added REF**135: VIA-0.3, JueVias:VIA-0.3, F.Cu at (105.0, 115.0)
- added REF**141: VIA-0.3, JueVias:VIA-0.3, F.Cu at (110.0, 95.0)
- added REF**145: VIA-0.3, JueVias:VIA-0.3, F.Cu at (110.0, 115.0)
- added REF**151: VIA-0.3, JueVias:VIA-0.3, F.Cu at (115.0, 95.0)
- added REF**153: VIA-0.3, JueVias:VIA-0.3, F.Cu at (115.0, 105.0)
- added REF**155: VIA-0.3, JueVias:VIA-0.3, F.Cu at (115.0, 115.0)
- added REF**161: VIA-0.3, JueVias:VIA-0.3, F.Cu at (120.0, 95.0)
- added REF**163: VIA-0.3, JueVias:VIA-0.3, F.Cu at (120.0, 105.0)
- added REF**165: VIA-0.3, JueVias:VIA-0.3, F.Cu at (120.0, 115.0)
- added REF**171: VIA-0.3, JueVias:VIA-0.3, F.Cu at (125.0, 95.0)
- added REF**172: VIA-0.3, JueVias:VIA-0.3, F.Cu at (125.0, 100.0)
- added REF**173: VIA-0.3, JueVias:VIA-0.3, F.Cu at (125.0, 105.0)
- added REF**175: VIA-0.3, JueVias:VIA-0.3, F.Cu at (125.0, 115.0)
- added REF**181: VIA-0.3, JueVias:VIA-0.3, F.Cu at (130.0, 95.0)
- added REF**185: VIA-0.3, JueVias:VIA-0.3, F.Cu at (130.0, 115.0)
- added REF**191: VIA-0.3, JueVias:VIA-0.3, F.Cu at (135.0, 95.0)
- added REF**192: VIA-0.3, JueVias:VIA-0.3, F.Cu at (135.0, 100.0)
- added REF**194: VIA-0.3, JueVias:VIA-0.3, F.Cu at (135.0, 110.0)
- added REF**195: VIA-0.3, JueVias:VIA-0.3, F.Cu at (135.0, 115.0)
Other:
- rule pad_to_mask_clearance: 0.127 -> 0.0762
