File: ERA-6SM+/ERA-6SM+.sch (KiCad schematic (older format))
At the start: 9 parts, among them P1 CONN_01X02, U1 ERA-6+, X1 SMA-F, X2 SMA-F

Commit message: ERA-6SM+: Changed from 12V supply to 10V
Parts:
- R1: value 100 / 1W -> 69.8 / 0.5W
Changed lines of the file:
@@
 P 6700 2500
 F 0 "R1" V 6600 2500 50  0000 C CNN
-F 1 "100 / 1W" V 6800 2500 50  0000 C CNN
+F 1 "69.8 / 0.5W" V 6800 2500 50  0000 C CNN
 F 2 "Resistors_SMD:R_1206" V 6630 2500 50  0001 C CNN
 F 3 "" H 6700 2500 50  0000 C CNN
